File: Hardware/Third_Year_Project_ele21zy.kicad_pcb (KiCad board)
At the start: 2 copper layers, 40 x 60 mm, 8 parts, among them J1 826926-5, J2 826926-5, J3 826926-5, J4 826926-5, J5 826926-5, J6 501876-2640

Commit message: update hardware
Parts:
- F1: value 0683G4000-01 -> 0686F2000-01; footprint 0683G4000-01:FUSE_0683G4000-01 -> 0686F2000-01:FUSC1608X60N
- R1: footprint Resistor_THT:R_Axial_DIN0204_L3.6mm_D1.6mm_P7.62mm_Horizontal -> KiCad:RESAD1050W45L330D180
- moved J4 11.0 mm to (129.0, 95.0), turned to -90 degrees
- moved R1 4.81 mm to (143.0, 96.0), turned to 90 degrees
- moved F1 3.24 mm to (143.0, 82.2)
- moved J2 1.02 mm to (139.0, 72.0)
Connections:
- J4 pad 5: CELL_14_Negative -> unconnected-(J4-Pad5)
- J5 pad 1: CELL_14_Negative -> CELL_1_Negative
- J5 pad 2: ISENSE_N -> CELL_1_Negative
- J5 pad 3: unconnected-(J5-Pad3) -> ISENSE_N
- J5 pad 4: GND -> unconnected-(J5-Pad4)
- J5 pad 5: unconnected-(J5-Pad5) -> GND
- J6 pad 12: CELL_14_Negative -> CELL_1_Negative
- R1 pad 1: ISENSE_N -> CELL_1_Negative
- R1 pad 2: CELL_14_Negative -> ISENSE_N
Routing:
- net CELL_14_Negative: track 56.5 -> 0.00 mm
- net CELL_1_Negative: track 0.00 -> 39.6 mm
- net CELL_11: track 19.1 -> 30.5 mm
- net CELL_13: track 29.8 -> 22.4 mm
- net CELL_14: track 20.8 -> 13.5 mm
- net GND: track 64.1 -> 70.2 mm
- net CELL_12: track 11.5 -> 17.4 mm
- net CELL_7: track 48.9 -> 51.7 mm
- net ISENSE_N: track 18.7 -> 21.2 mm
- net CELL_9: track 40.5 -> 41.9 mm
- net CELL_5: track 61.2 -> 62.6 mm
- net CELL_2: track 43.1 -> 44.4 mm
- net CELL_4: track 44.4 -> 45.3 mm
Other:
- board text added: "CT1"
- board text added: "CT10"
- board text added: "CT11"
- board text added: "CT12"
- board text added: "CT13"
- board text added: "CT14"
- board text added: "CT2"
- board text added: "CT3"
- board text added: "CT4"
- board text added: "CT5"
- board text added: "CT6"
- board text added: "CT7"
- board text added: "CT8"
- board text added: "CT9"
- board text added: "Cell_1_Neg"
- board text removed: "C1"
- board text removed: "C10"
- board text removed: "C11"
- board text removed: "C12"
- board text removed: "C13"
- board text removed: "C14"
- board text removed: "C2"
- board text removed: "C3"
- board text removed: "C4"
- board text removed: "C5"
- board text removed: "C6"
- board text removed: "C7"
- board text removed: "C8"
- board text removed: "C9"
- board text removed: "REF"

Commit message: update hardware
Parts:
- added J6: MC000048, MC000048:MC000048, F.Cu at (161.0, 72.0)
- added REF**: Symbol_HighVoltage_Type2_CopperTop_VerySmall, Symbol:Symbol_HighVoltage_Type2_CopperTop_VerySmall, F.Cu at (180.0, 74.0)
- added SW1: L102011MS02Q, L102011MS02Q:L102011MS02Q, F.Cu at (144.0, 92.0)
- added TP1: 930224100, 930224100:930224100, F.Cu at (168.0, 122.0)
- added TP2: 930224100, 930224100:930224100, F.Cu at (177.0, 122.0)
- F1: value 0686F2000-01 -> 39212000440; footprint 0686F2000-01:FUSC1608X60N -> 39212000440:39213150440_1
- J1, J2, J3, J4, J5: footprint 826926-5:TE_826926-5 -> 2212S-05SG-85:RHDR5W74P0X254_1X5_1320X250X850P
- R1: value 0.1 -> 43FR10E; footprint KiCad:RESAD1050W45L330D180 -> 43FR10E:RESAD3750W90L1510D560
- moved R1 38.8 mm to (172.0, 70.2), turned to -90 degrees
- moved F1 21.1 mm to (146.6, 103.0), turned to 0 degrees
- moved J5 3.80 mm to (161.0, 92.2)
- moved J1 2.98 mm to (161.0, 108.0)
- renumbered J6 to J7
Connections:
- F1 pad 1: ISENSE_N -> Net-(F1-Pad1)
- F1 pad 2: GND -> ISENSE_P
- J4 pad 4: CELL_14 -> unconnected-(J4-Pad4)
- J4 pad 5: unconnected-(J4-Pad5) -> CELL_14
- J5 pad 1: CELL_1_Negative -> unconnected-(J5-Pad1)
- J5 pad 2: CELL_1_Negative -> unconnected-(J5-Pad2)
- J5 pad 3: ISENSE_N -> ISENSE_P
- R1 pad 1: CELL_1_Negative -> ISENSE_P
- R1 pad 2: ISENSE_N -> GND
Routing:
- net CELL_1_Negative: track 39.6 -> 99.5 mm
- net CELL_14: track 13.5 -> 59.4 mm
- net ISENSE_P: track 0.00 -> 45.3 mm
- net CELL_3: track 92.4 -> 136.9 mm
- net CELL_1: track 79.1 -> 119.3 mm
- net ISENSE_N: track 21.2 -> 0.00 mm
- net Net-(F1-Pad1): track 0.00 -> 11.0 mm
- net GND: track 70.2 -> 75.9 mm
- net NTC4: track 15.4 -> 14.5 mm
- net NTC6: track 8.65 -> 7.86 mm
- net NTC5: track 12.2 -> 11.5 mm
- net NTC3: track 18.8 -> 18.2 mm
Other:
- board size 40 x 60 mm -> 62.8 x 62.8 mm
- board text added: "BATT Neg"
- board text added: "BATT Pos"
- board text added: "X"
