File: Hardware/Third_Year_Project_ele21zy.kicad_sch (KiCad schematic)
At the start: 8 parts, among them J1 826926-5, J2 826926-5, J3 826926-5, J4 826926-5, J5 826926-5, J6 501876-2640

Commit message: update hardware
Parts:
- removed F1: 0683G4000-01, FUSE_0683G4000-01, symbol 0683G4000-01:0683G4000-01
- added F1: 0686F2000-01, FUSC1608X60N, symbol 0686F2000-01:0686F2000-01
- R1: footprint Resistor_THT:R_Axial_DIN0204_L3.6mm_D1.6mm_P7.62mm_Horizontal -> RESAD1050W45L330D180; symbol Device:R -> RSMOA0318FAOHR100:RSMOA0318FAOHR100; Manufacturer_Name (none) -> RS Components; Manufacturer_Part_Number (none) -> RSMOA0318FAOHR100
Connections:
- net GND: now also J5.5, F1.2; no longer J5.4
- net ISENSE_N: now also J5.3, R1.2, F1.1; no longer J5.2, R1.1
- net CELL_14_Negative renamed CELL_1_Negative
- net CELL_1_Negative: now also J5.2, R1.1; no longer J4.5, R1.2

Commit message: update hardware
Parts:
- removed F1: 0686F2000-01, FUSC1608X60N, symbol 0686F2000-01:0686F2000-01
- removed R1: 0.1, RESAD1050W45L330D180, symbol RSMOA0318FAOHR100:RSMOA0318FAOHR100
- added F1: 39212000440, 39213150440_1, symbol 39212000440:39212000440
- added J6: MC000048, MC000048, symbol MC000048:MC000048
- added R1: 43FR10E, RESAD3750W90L1510D560, symbol 43FR10E:43FR10E
- added SW1: L102011MS02Q, L102011MS02Q:L102011MS02Q, symbol Switch:SW_SPDT
- added TP1, TP2: 930224100, 930224100, symbol 930224100:930224100
- J1, J2, J3, J4, J5: footprint TE_826926-5 -> 2212S-05SG-85:RHDR5W74P0X254_1X5_1320X250X850P; symbol 826926-5:826926-5 -> 2212S-05SG-85:2212S-05SG-85; Height (none) -> 8.5; Manufacturer_Name (none) -> MULTICOMP; Manufacturer_Part_Number (none) -> 2212S-05SG-85
- renumbered J6 to J7
Connections:
- net CELL_14: now also J4.5, TP1.1, TP1.2; no longer J4.4
- net CELL_1_Negative: now also J6.2, SW1.2 (B), TP2.1, TP2.2; no longer J5.1, J5.2
- net GND: now also J6.1, R1.2
- net ISENSE_N renamed ISENSE_P
- net ISENSE_P: now also F1.2, R1.1
- new net: F1.1, SW1.1 (A)
- no-connect marks 3 -> 6
Other:
- moved on the sheet: J7
